Commit message: [pr2_urdf] adjusted values for torso lift joint

File: resources/pr2.urdf (robot description, URDF)
Before this commit: robot pr2, 88 links, 87 joints
Joints:
- joint torso_lift_joint: limit lower=0. upper=0.33 effort=1000 velocity=0.13 -> lower=0.0 upper=0.33 effort=10000 velocity=0.013
